File: PCB/Rojko.kicad_pcb (KiCad board)
At the start: 2 copper layers, 20 x 24 mm, 33 parts, among them IC1 STM32L051C8T6, IC2 BQ25186DLHR, IC3 AP63203WU-7, J1 AYF-531035, J4 +, J5 -, J6 AYF-531035, SW1 SW_MEC_5G, U1 RYB080I, Y1 32,768k

Commit message: adda
Parts:
- removed C1, C6: 1uF, Capacitor_SMD:C_0201_0603Metric
- removed C10, C8, C9: 100n, Capacitor_SMD:C_0201_0603Metric
- removed C2: 100nF, Capacitor_SMD:C_0201_0603Metric
- removed C3: 10uF, Capacitor_SMD:C_0201_0603Metric
- removed C4, C7: 10pF, Capacitor_SMD:C_0201_0603Metric
- removed C5: 10nF, Capacitor_SMD:C_0201_0603Metric
- removed FB1: FerriteBead, Resistor_SMD:R_0805_2012Metric
- removed FB2: FerriteBead, Resistor_SMD:R_0201_0603Metric
- removed IC1: STM32L051C8T6, Package_QFP:LQFP-48_7x7mm_P0.5mm
- removed R1: 10k, Resistor_SMD:R_0201_0603Metric
- removed SW1: SW_MEC_5G, CUSTOM:SWITCH small
- removed U1: RYB080I, RYB080l:RYB080i
- removed Y1: 32,768k, Crystal:Crystal_SMD_3215-2Pin_3.2x1.5mm
- added AE1: PCB antenna, RF_Antenna:Texas_SWRA117D_2.4GHz_Right, B.Cu at (175.2, 129.7)
- added C20: 1uF, Capacitor_SMD:C_0201_0603Metric, F.Cu at (174.8, 88.2)
- added C21: 100n, Capacitor_SMD:C_0201_0603Metric, F.Cu at (217.9, 123.3)
- added C22: 4.7uF, Capacitor_SMD:C_0201_0603Metric, F.Cu at (174.8, 91.8)
- added C23: 10nF, Capacitor_SMD:C_0201_0603Metric, F.Cu at (174.8, 93.5)
- added C24: 1uF, Capacitor_SMD:C_0201_0603Metric, F.Cu at (174.8, 95.2)
- added C25: 100n, Capacitor_SMD:C_0201_0603Metric, F.Cu at (174.8, 97.0)
- added C26: 100n, Capacitor_SMD:C_0201_0603Metric, F.Cu at (174.8, 98.8)
- added C27: 4.7uF, Capacitor_SMD:C_0201_0603Metric, F.Cu at (177.2, 86.5)
- added C28: 0.8pF, Capacitor_SMD:C_0201_0603Metric, F.Cu at (224.4, 120.7)
- added C29: 100nF, Capacitor_SMD:C_0201_0603Metric, F.Cu at (177.2, 90.0)
- added C30: 10pF, Capacitor_SMD:C_0201_0603Metric, F.Cu at (177.2, 91.8)
- added C31: 10pF, Capacitor_SMD:C_0201_0603Metric, F.Cu at (177.2, 93.5)
- added C32: 100n, Capacitor_SMD:C_0201_0603Metric, F.Cu at (177.2, 95.2)
- added C33: 100n, Capacitor_SMD:C_0201_0603Metric, F.Cu at (177.2, 97.0)
- added C34: 100n, Capacitor_SMD:C_0201_0603Metric, F.Cu at (177.2, 98.8)
- added C35: 0.3pF, Capacitor_SMD:C_0201_0603Metric, F.Cu at (224.4, 121.6)
- added FB3: 30-120Ohm@100Mhz, Resistor_SMD:R_0805_2012Metric, F.Cu at (194.6, 101.2)
- added FL1: DLF162500LT-5028A1, DLF162500LT-5028A1:DLF162500LT5028A1, F.Cu at (230.9, 128.6)
- added IC4: STM32WB35CEU6A, STM32WB35CEU6A:QFN50P700X700X60-49N-D, F.Cu at (169.6, 119.5)
- added J2: +, CUSTOM:SMD pad, F.Cu at (190.8, 94.3)
- added J3: -, CUSTOM:SMD pad, F.Cu at (190.8, 97.4)
- added L2: 10uH, Inductor_SMD:L_0603_1608Metric, F.Cu at (177.8, 110.2)
- added L3: 2.7nH, Inductor_SMD:L_0201_0603Metric, F.Cu at (223.1, 121.1)
- added R3: 10k, Resistor_SMD:R_0201_0603Metric, F.Cu at (179.7, 91.8)
- added SW3: SW_MEC_5G, CUSTOM:SWITCH small, F.Cu at (173.4, 110.3)
- added Y2: Crystal_GND24, Crystal:Crystal_SMD_2016-4Pin_2.0x1.6mm, F.Cu at (194.4, 97.9)
- added Y3: 32,768k, Crystal:Crystal_SMD_3215-2Pin_3.2x1.5mm, F.Cu at (194.9, 94.4)
- C12, C14, C15, C16, C17, C18, IC3, J1: moved to F.Cu
- L1: footprint Inductor_SMD:L_0805_2012Metric -> Inductor_SMD:L_0201_0603Metric; moved to F.Cu
- moved C14 71.6 mm to (211.5, 124.5), turned to -90 degrees
- moved J1 70.4 mm to (210.2, 122.7), turned to -90 degrees
- moved C15 68.6 mm to (209.0, 124.1), turned to -90 degrees
- moved C12 66.4 mm to (208.0, 123.5), turned to 90 degrees
- moved IC2 46.2 mm to (198.5, 107.0), turned to 180 degrees
- moved J4 40.5 mm to (190.8, 100.5), turned to 0 degrees
- moved IC3 40.2 mm to (192.1, 108.3)
- moved J5 39.5 mm to (190.8, 103.6), turned to 0 degrees
- moved J6 31.3 mm to (185.0, 99.0), turned to 0 degrees
- moved L1 25.9 mm to (179.7, 88.2)
- moved C11 19.1 mm to (172.3, 86.5)
- moved C18 19.0 mm to (172.3, 98.8)
- moved C19 19.0 mm to (174.8, 86.5), turned to 0 degrees
- moved C13 17.6 mm to (172.3, 90.0), turned to 0 degrees
- moved C16 15.3 mm to (172.3, 95.2), turned to 0 degrees
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Connections:
- J6 pad 1: unconnected-(J6-Pad1) -> PROG_SWDIO
- J6 pad 10: GND -> unconnected-(J6-Pad10)
- J6 pad 3: unconnected-(J6-Pad3) -> +3.3V
- J6 pad 4: +3.3V -> GND
- J6 pad 5: unconnected-(J6-Pad5) -> PROG_SWCLK
- J6 pad 6: PROG_SWDIO -> unconnected-(J6-Pad6)
- J6 pad 7: unconnected-(J6-Pad7) -> PROG_SWO
- J6 pad 8: PROG_SWCLK -> unconnected-(J6-Pad8)
- J6 pad 9: unconnected-(J6-Pad9) -> GND
Routing:
- net GND: track 109.2 -> 6.53 mm, vias 1 -> 0
- net +3.3V: track 47.3 -> 5.82 mm
- net BAT_SCL: track 25.6 -> 0.00 mm, vias 2 -> 0
- net BAT_SDA: track 23.8 -> 0.00 mm, vias 2 -> 0
- net BAT_INT: track 20.2 -> 0.00 mm, vias 2 -> 0
- net BAT_GPO: track 19.9 -> 0.00 mm, vias 2 -> 0
- net BAT_CE: track 18.7 -> 0.00 mm, vias 2 -> 0
- net +5V: track 10.9 -> 0.00 mm, vias 1 -> 0
- net DISP_MOSI: track 0.00 -> 6.79 mm, vias 0 -> 2
- net DISP_SCK: track 8.91 -> 2.40 mm, vias 1 -> 0
- net Net-(IC1-NRST): track 6.40 -> 0.00 mm
- net Net-(IC2-BAT): track 6.25 -> 0.00 mm
- net Net-(IC2-TS/MR): track 4.88 -> 0.00 mm
- net Net-(C3-Pad2): track 4.87 -> 0.00 mm
- net DISP_SCS : track 7.96 -> 3.19 mm, vias 1 -> 0
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Other:
- outline, holes or cut-outs redrawn

Commit message: plostica
Parts:
- removed C11: 10uF, Capacitor_SMD:C_0201_0603Metric
- removed C13, C19: 1uF, Capacitor_SMD:C_0201_0603Metric
- removed IC2: BQ25186DLHR, BQ25186DLHR:SON40P220X200X80-11N
- removed J2, J4: +, CUSTOM:SMD pad
- removed J3, J5: -, CUSTOM:SMD pad
- C16, C17, C18, C20, C23, C24, C27, C28, C30, C31, C32, C33, C34, C35, FB3, FL1, J1, L1, L2, L3, R3, Y2: moved to B.Cu
- moved FL1 134.2 mm to (99.5, 101.1)
- moved C35 128.5 mm to (98.1, 98.0)
- moved C28 127.0 mm to (99.4, 98.6), turned to 90 degrees
- moved L3 126.9 mm to (98.1, 99.1), turned to 180 degrees
- moved C14 117.0 mm to (99.6, 90.2), turned to 180 degrees
- moved C15 114.3 mm to (99.6, 91.1), turned to 180 degrees
- moved J1 113.6 mm to (100.9, 91.8), turned to 90 degrees
- moved C12 112.9 mm to (99.6, 92.0), turned to 0 degrees
- moved C21 112.4 mm to (108.8, 96.1)
- moved FB3 95.8 mm to (100.0, 86.1), turned to 180 degrees
- moved Y3 95.1 mm to (100.1, 87.6), turned to 180 degrees
- moved Y2 84.8 mm to (109.8, 94.4), turned to -90 degrees
- moved IC3 79.3 mm to (114.1, 93.9), turned to 180 degrees
- moved J6 79.1 mm to (107.1, 85.8), turned to 180 degrees
- moved C30 78.2 mm to (99.2, 87.6), turned to 180 degrees
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Routing:
- net GND: track 6.53 -> 61.3 mm, vias 0 -> 4
- net +3.3V: track 5.82 -> 34.5 mm, vias 0 -> 6
- net Net-(IC4-NRST): track 0.00 -> 12.2 mm
- net Net-(IC4-RF1): track 0.62 -> 12.6 mm, vias 0 -> 1
- net Net-(IC4-PC15-OSC32_OUT): track 0.00 -> 5.54 mm, vias 0 -> 1
- net +3.3VA: track 7.81 -> 13.3 mm
- net Net-(IC4-VFBSMPS): track 0.00 -> 5.52 mm, vias 0 -> 1
- net Net-(AE1-A): track 4.08 -> 8.60 mm, vias 1 -> 0
- net DISP_VCOM: track 4.54 -> 8.19 mm, vias 0 -> 1
- net Net-(IC4-VLXSMPS): track 0.00 -> 3.45 mm, vias 0 -> 1
- net Net-(IC4-PC14-OSC32_IN): track 0.00 -> 2.77 mm, vias 0 -> 1
- net DISP_ON/OFF: track 8.00 -> 10.7 mm, vias 0 -> 1
- net Net-(IC4-OSC_OUT): track 0.00 -> 2.51 mm, vias 0 -> 1
- net PROG_SWDIO: track 0.00 -> 2.25 mm
- net PROG_SWO: track 0.00 -> 2.10 mm
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- added copper zone on F.Cu, net GND
Other:
- board size 20 x 24 mm -> 20 x 20 mm

Commit message: dwa
Parts:
- removed FL1: DLF162500LT-5028A1, DLF162500LT-5028A1:DLF162500LT5028A1
- added C1: 100nF, Capacitor_SMD:C_0201_0603Metric, F.Cu at (113.8, 100.4)
- added C2: 100nF, Capacitor_SMD:C_0201_0603Metric, F.Cu at (105.6, 85.9)
- added SW1: SW_MEC_5G, CUSTOM:Switch small but not that small, F.Cu at (116.1, 100.7)
- added SW2: SW_MEC_5G, CUSTOM:Switch small but not that small, F.Cu at (106.4, 83.8)
- AE1, C20, C23, C24, C27, C28, C30, C31, C32, C33, C34, C35, L1, L3, R3: moved to F.Cu
- C16, C17, C18: footprint Capacitor_SMD:C_0201_0603Metric -> Capacitor_SMD:C_0805_2012Metric
- moved C35 12.1 mm to (110.1, 96.9)
- moved L3 10.6 mm to (108.5, 96.9), turned to 0 degrees
- moved C28 9.47 mm to (108.5, 96.1), turned to 0 degrees
- moved C17 7.14 mm to (115.8, 87.1), turned to -90 degrees
- moved J6 6.38 mm to (113.4, 86.5), turned to 90 degrees
- moved AE1 5.17 mm to (109.8, 98.1), turned to 180 degrees
- moved C27 3.74 mm to (112.3, 85.5)
- moved L1 2.31 mm to (115.5, 90.6), turned to 0 degrees
- moved C30 2.17 mm to (99.7, 89.7), turned to 90 degrees
- moved C14 2.15 mm to (99.6, 92.4)
- moved C12 2.15 mm to (99.6, 94.2)
- moved C15 2.15 mm to (99.6, 93.3)
- moved J1 2.15 mm to (100.9, 94.0)
- moved C31 2.03 mm to (101.0, 89.6)
- moved C20 2.00 mm to (102.9, 84.6), turned to -90 degrees
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Connections:
- AE1 pad 1: Net-(AE1-A) -> /RF
- C35 pad 1: Net-(FL1-IN) -> /RF
- IC4 pad 28: unconnected-(IC4-PB0-Pad28) -> Net-(IC4-PB0)
- IC4 pad 29: BAT_GPO -> unconnected-(IC4-PB1-Pad29)
- IC4 pad 45: unconnected-(IC4-PB5-Pad45) -> Net-(IC4-PB5)
- L3 pad 2: Net-(FL1-IN) -> /RF
Routing:
- net +3.3V: track 34.5 -> 52.9 mm, vias 6 -> 8
- net Net-(IC4-PB0): track 0.00 -> 13.4 mm, vias 0 -> 2
- net GND: track 61.3 -> 73.1 mm, vias 4 -> 15
- net Net-(IC4-RF1): track 12.6 -> 2.19 mm, vias 1 -> 0
- net Net-(AE1-A): track 8.60 -> 0.00 mm
- net PROG_SWO: track 2.10 -> 10.6 mm, vias 0 -> 2
- net DISP_MOSI: track 8.71 -> 0.92 mm
- net +3.3VA: track 13.3 -> 20.4 mm, vias 2 -> 3
- net Net-(IC4-PB5): track 0.00 -> 6.11 mm
- net PROG_SWCLK: track 2.10 -> 7.73 mm, vias 0 -> 2
- net PROG_SWDIO: track 2.25 -> 6.08 mm
- net DISP_ON/OFF: track 10.7 -> 7.18 mm, vias 1 -> 2
- net Net-(FL1-IN): track 3.51 -> 0.00 mm
- net DISP_VCOM: track 8.19 -> 4.80 mm
- net Net-(C17-Pad2): track 0.99 -> 3.28 mm, vias 0 -> 1
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- added copper zone on B.Cu, net GND
Other:
- board size 20 x 20 mm -> 20 x 20.9 mm
