File: PCB/Rojko.kicad_sch (KiCad schematic)
At the start: 30 parts, among them IC1 STM32L051C8T6, IC2 BQ25186DLHR, IC3 AP63203WU-7, J1 Conn_01x10_Socket, J2 Conn_01x10_Socket, SW1 SW_MEC_5G, Y1 32,768k

Commit message: ble add
Parts:
- added U1: RYB080I, symbol RYB080l:RYB080i
Connections:
- net +3.3V: now also U1.12 (VDD), U1.13 (VDD)
- net GND: now also U1.1 (GND), U1.16 (GND), U1.22 (GND), U1.3 (GND), U1.7 (GND)
- new net BLE_NRST: U1.15 (RESET_N)
- new net BLE_RX: U1.4 (DIO0/WAKE_UP), U1.5 (DIO1/RXD)
- new net BLE_TX: U1.6 (DIO2/TXD)

Commit message: dsa
Parts:
- removed BT1, BT2: 3.7V 30mA, symbol Device:Battery_Cell
- removed C16, C17: 1uF, symbol Device:C
- removed C18: 0.1uF, symbol Device:C
- removed J1, J2: Conn_01x10_Socket, symbol Connector:Conn_01x10_Socket
- added C12: 0.1uF, Capacitor_SMD:C_0201_0603Metric, symbol Device:C
- added C14, C15: 1uF, Capacitor_SMD:C_0201_0603Metric, symbol Device:C
- added C3: 10uF, Capacitor_SMD:C_0201_0603Metric, symbol Device:C
- added FB2: FerriteBead, Resistor_SMD:R_0201_0603Metric, symbol Device:FerriteBead
- added J1, J6: AYF-531035, AYF-531035:AYF531035, symbol AYF-531035:AYF-531035
- added J2, J4: +, CUSTOM:SMD pad, symbol Connector:Conn_01x01_Socket
- added J3, J5: -, CUSTOM:SMD pad, symbol Connector:Conn_01x01_Socket
- C1: renamed from C15; footprint (none) -> Capacitor_SMD:C_0201_0603Metric
- C10: renamed from C14; footprint (none) -> Capacitor_SMD:C_0201_0603Metric
- C11: renamed from C12; footprint (none) -> Capacitor_SMD:C_0201_0603Metric
- C13, C5, C6: footprint (none) -> Capacitor_SMD:C_0201_0603Metric
- C16: renamed from C10; footprint (none) -> Capacitor_SMD:C_0201_0603Metric
- C17: renamed from C8; footprint (none) -> Capacitor_SMD:C_0201_0603Metric
- C18: renamed from C9; footprint (none) -> Capacitor_SMD:C_0201_0603Metric
- C19: renamed from C11; footprint (none) -> Capacitor_SMD:C_0201_0603Metric
- C2: renamed from C4; footprint (none) -> Capacitor_SMD:C_0201_0603Metric
- C4: renamed from C3; footprint (none) -> Capacitor_SMD:C_0201_0603Metric
- C7: renamed from C2; footprint (none) -> Capacitor_SMD:C_0201_0603Metric
- C8: renamed from C1; footprint (none) -> Capacitor_SMD:C_0201_0603Metric
- C9: renamed from C7; footprint (none) -> Capacitor_SMD:C_0201_0603Metric
- FB1: footprint (none) -> Resistor_SMD:R_0805_2012Metric
- IC1: footprint Package_CSP:ST_WLCSP-36_Die417 -> Package_QFP:LQFP-48_7x7mm_P0.5mm
- IC2: footprint SON40P220X200X80-11N -> BQ25186DLHR:SON40P220X200X80-11N
- IC3: footprint AP63203WU7 -> AP63203WU-7:AP63203WU7
- L1: footprint (none) -> Inductor_SMD:L_0805_2012Metric
- R1: footprint (none) -> Resistor_SMD:R_0201_0603Metric
- SW1: footprint (none) -> CUSTOM:SWITCH small
- U1: footprint (none) -> RYB080l:RYB080i
- Y1: footprint (none) -> Crystal:Crystal_SMD_3215-2Pin_3.2x1.5mm
Connections:
- net +3.3V: now also C14.1, FB2.2, J1.7, J1.8, J6.4; no longer U1.12 (VDD), U1.13 (VDD)
- net +3.3VA: now also C15.1, J1.6
- net DISP_MOSI: now also J1.2
- net DISP_ON/OFF: now also C12.2, J1.5
- net DISP_SCK: now also J1.1
- net DISP_SCS : now also J1.3
- net DISP_VCOM: now also J1.4
- net GND: now also C3.1, J6.10
- net PROG_SWCLK: now also J6.8
- net PROG_SWDIO: now also J6.6
- net at C13.1, IC2.2 (BAT): now also J2.1 (Pin_1), J4.1 (Pin_1)
- net at IC2.6 (TS/MR): now also J3.1 (Pin_1), J5.1 (Pin_1)
- new net: C3.2, FB2.1, U1.12 (VDD), U1.13 (VDD)
- new net: C12.1, C14.2, C15.2, J1.10, J1.9
Other:
- note added: "2x 3,7V Li-Ion 30mA"

Commit message: zmena chipu
Parts:
- removed C1, C6: 1uF, Capacitor_SMD:C_0201_0603Metric, symbol Device:C
- removed C10, C8, C9: 100n, Capacitor_SMD:C_0201_0603Metric, symbol Device:C
- removed C2: 100nF, Capacitor_SMD:C_0201_0603Metric, symbol Device:C
- removed C3: 10uF, Capacitor_SMD:C_0201_0603Metric, symbol Device:C
- removed C4, C7: 10pF, Capacitor_SMD:C_0201_0603Metric, symbol Device:C
- removed C5: 10nF, Capacitor_SMD:C_0201_0603Metric, symbol Device:C
- removed FB1: FerriteBead, Resistor_SMD:R_0805_2012Metric, symbol Device:FerriteBead
- removed FB2: FerriteBead, Resistor_SMD:R_0201_0603Metric, symbol Device:FerriteBead
- removed IC1: STM32L051C8T6, Package_QFP:LQFP-48_7x7mm_P0.5mm, symbol STM32L051C8T6:STM32L051C8T6
- removed R1: 10k, Resistor_SMD:R_0201_0603Metric, symbol Device:R
- removed SW1: SW_MEC_5G, CUSTOM:SWITCH small, symbol Switch:SW_MEC_5G
- removed U1: RYB080I, RYB080l:RYB080i, symbol RYB080l:RYB080i
- removed Y1: 32,768k, Crystal:Crystal_SMD_3215-2Pin_3.2x1.5mm, symbol Device:Crystal
- added AE1: PCB antenna, RF_Antenna:Texas_SWRA117D_2.4GHz_Right, symbol Device:Antenna_Shield
- added C20, C24: 1uF, Capacitor_SMD:C_0201_0603Metric, symbol Device:C
- added C21: 100n, symbol Device:C_Polarized
- added C22, C27: 4.7uF, Capacitor_SMD:C_0201_0603Metric, symbol Device:C
- added C23: 10nF, Capacitor_SMD:C_0201_0603Metric, symbol Device:C
- added C25, C26, C32, C33, C34: 100n, Capacitor_SMD:C_0201_0603Metric, symbol Device:C
- added C28: 0.8pF, symbol Device:C
- added C29: 100nF, Capacitor_SMD:C_0201_0603Metric, symbol Device:C
- added C30, C31: 10pF, Capacitor_SMD:C_0201_0603Metric, symbol Device:C
- added C35: 0.3pF, symbol Device:C
- added FB3: 30-120Ohm@100Mhz, Resistor_SMD:R_0805_2012Metric, symbol Device:FerriteBead
- added FL1: DLF162500LT-5028A1, DLF162500LT5028A1, symbol DLF162500LT-5028A1:DLF162500LT-5028A1
- added IC4: STM32WB35CEU6A, QFN50P700X700X60-49N-D, symbol STM32WB35CEU6A:STM32WB35CEU6A
- added L2: 10uH, symbol Device:L
- added L3: 2.7nH, symbol Device:L
- added R3: 10k, Resistor_SMD:R_0201_0603Metric, symbol Device:R
- added SW3: SW_MEC_5G, CUSTOM:SWITCH small, symbol Switch:SW_MEC_5G
- added Y2: Crystal_GND24, symbol Device:Crystal_GND24
- added Y3: 32,768k, Crystal:Crystal_SMD_3215-2Pin_3.2x1.5mm, symbol Device:Crystal
Connections:
- net +3.3V: now also C20.1, C25.1, C26.1, C27.1, C32.1, C33.1, C34.1, FB3.1, IC4.1 (VBAT), IC4.20 (VDD_1), IC4.34 (VDDSMPS), IC4.35 (VDD_2), IC4.40 (VDDUSB), IC4.48 (VDD_3)
- net +3.3VA: now also C23.1, C24.1, FB3.2, IC4.8 (VDDA)
- net BAT_CE: now also IC4.46 (PB6)
- net BAT_GPO: now also IC4.45 (PB5)
- net BAT_INT: now also IC4.47 (PB7)
- net BAT_SCL: now also IC4.5 (PB8)
- net BAT_SDA: now also IC4.6 (PB9)
- net DISP_MOSI: now also IC4.16 (PA7)
- net DISP_ON/OFF: now also IC4.15 (PA6)
- net DISP_SCK: now also IC4.10 (PA1)
- net DISP_SCS : now also IC4.13 (PA4)
- net DISP_VCOM: now also IC4.14 (PA5)
- net GND: now also AE1.2 (Shield), C20.2, C21.2, C22.2, C23.2, C24.2, C25.2, C26.2, C27.2, C28.2, C29.1, C30.1, C31.1, C32.2, C33.2, C34.2, C35.2, FL1.2 (GND_1), FL1.4 (GND_2), IC4.22 (VSSRF), IC4.32 (VSSSMPS), R3.1, SW3.1 (A), SW3.2 (A), Y2.2, Y2.4
- net PROG_SWCLK: now also IC4.41 (PA14)
- net PROG_SWDIO: now also IC4.39 (PA13)
- new net: C21.1, IC4.23 (VDDRF)
- new net: C35.1, FL1.1 (IN), L3.2
- new net: AE1.1 (A), FL1.3 (OUT)
- new net: C31.2, IC4.2 (PC14-OSC32_IN), Y3.2
- new net: C22.1, IC4.31 (VFBSMPS), L2.2
- new net: C30.2, IC4.3 (PC15-OSC32_OUT), Y3.1
- new net: C29.2, IC4.7 (NRST), SW3.3 (B), SW3.4 (B)
- new net: IC4.33 (VLXSMPS), L2.1
- new net: IC4.4 (PH3-BOOT0), R3.2
- new net: IC4.25 (OSC_IN), Y2.1
- new net: IC4.24 (OSC_OUT), Y2.3
- new net: C28.1, IC4.21 (RF1), L3.1
- new net PROG_SWO: IC4.43 (PB3)
Other:
- moved on the sheet: C12, C14, C15, J1, J6

Commit message: adda
Parts:
- C21, C28, C35: footprint (none) -> Capacitor_SMD:C_0201_0603Metric
- FL1: footprint DLF162500LT5028A1 -> DLF162500LT-5028A1:DLF162500LT5028A1
- IC4: footprint QFN50P700X700X60-49N-D -> STM32WB35CEU6A:QFN50P700X700X60-49N-D
- L1: footprint Inductor_SMD:L_0805_2012Metric -> Inductor_SMD:L_0201_0603Metric
- L2: footprint (none) -> Inductor_SMD:L_0603_1608Metric
- L3: footprint (none) -> Inductor_SMD:L_0201_0603Metric
- Y2: footprint (none) -> Crystal:Crystal_SMD_2016-4Pin_2.0x1.6mm
Connections:
- net +3.3V: now also J6.3; no longer J6.4
- net BAT_GPO: now also IC4.29 (PB1); no longer IC4.45 (PB5)
- net GND: now also J6.4, J6.9; no longer J6.10
- net PROG_SWCLK: now also J6.5; no longer J6.8
- net PROG_SWDIO: now also J6.1; no longer J6.6
- net PROG_SWO: now also J6.7
Other:
- moved on the sheet: R3

Commit message: plostica
Parts:
- removed C11: 10uF, Capacitor_SMD:C_0201_0603Metric, symbol Device:C
- removed C13, C19: 1uF, Capacitor_SMD:C_0201_0603Metric, symbol Device:C
- removed IC2: BQ25186DLHR, BQ25186DLHR:SON40P220X200X80-11N, symbol BQ25186DLHR:BQ25186DLHR
- removed J2, J4: +, CUSTOM:SMD pad, symbol Connector:Conn_01x01_Socket
- removed J3, J5: -, CUSTOM:SMD pad, symbol Connector:Conn_01x01_Socket
Other:
- note removed: "2x 3,7V Li-Ion 30mA"

Commit message: dwa
Parts:
- removed FL1: DLF162500LT-5028A1, DLF162500LT-5028A1:DLF162500LT5028A1, symbol DLF162500LT-5028A1:DLF162500LT-5028A1
- added C1, C2: 100nF, Capacitor_SMD:C_0201_0603Metric, symbol Device:C
- added SW1, SW2: SW_MEC_5G, CUSTOM:Switch small but not that small, symbol Switch:SW_MEC_5G
- C16, C17, C18: footprint Capacitor_SMD:C_0201_0603Metric -> Capacitor_SMD:C_0805_2012Metric
Connections:
- net GND: now also C1.2, C2.1, SW1.3 (B), SW1.4 (B), SW2.1 (A), SW2.2 (A)
- net RF: now reaches C35.1, L3.2
- net RF: now also AE1.1 (A)
- net at IC4.28 (PB0): now also C1.1, SW1.1 (A), SW1.2 (A)
- net at IC4.45 (PB5): now also C2.2, SW2.3 (B), SW2.4 (B)
- net BAT_GPO: no longer names the net of IC4.29 (PB1)
Other:
- moved on the sheet: AE1, C22
